File: KiCad/Protopaja.kicad_pcb (KiCad board)
At the start: 2 copper layers, 49.5 x 61 mm, 81 parts, among them IC1 MCP73831T-2ATI_OT, IC2 BQ29733DSER, IC3 CP2102-GM, J1 USB_OTG, J2 B2B-PH-K-S(LF)(SN), J3 CONN_01X04, J4 CONN_01X08, Q1 CSD17575Q3, Q2 CSD17575Q3, Q3 PBSS4120T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

Commit message: Added the final report and updated KiCad files
Parts:
- added R19: R_0805_HandSoldering, Resistors_SMD:R_0805_HandSoldering, F.Cu at (158.1, 90.6)
- moved REF** 6.90 mm to (159.3, 83.4)
- moved REF** 2.05 mm to (155.8, 88.4)
Connections:
- IC1 pad 2: Net-(IC1-Pad2) -> GND
- R6 pad 2: Net-(IC1-Pad2) -> GND
Routing:
- net Net-(IC1-Pad2): track 10.3 -> 0.00 mm, vias 2 -> 0
- net /IO0: track 29.8 -> 33.2 mm
- net +3V3: track 159.8 -> 162.9 mm
- net /-BATT: track 41.9 -> 40.2 mm
- net Net-(IC2-Pad6): track 12.0 -> 12.6 mm, vias 2 -> 3
Other:
- net class Power: trace_width 0.7 -> 1
