File: KiCad/Protopaja.sch (KiCad schematic (older format))
At the start: 48 parts, among them IC1 MCP73831T-2ATI_OT, IC2 BQ29733DSER, IC3 CP2102-GM, J1 USB_OTG, J2 B2B-PH-K-S(LF)(SN), J3 CONN_01X04, J4 CONN_01X08, Q1 CSD17575Q3, Q2 CSD17575Q3, Q3 PBSS4120T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

Commit message: Added the final report and updated KiCad files
Parts:
- added R19: 10kΩ, symbol R_Small
Connections:
- net +3V3: now also R19.1
- net IO0: now also R19.2
Changed lines of the file:
@@
 Sheet 1 1
 Title "Futuwear V2"
-Date "2017-08-10"
-Rev "2.0"
+Date "2017-08-25"
+Rev "2.1"
 Comp "Protopaja"
 Comment1 "Drawn by Bruce Clayhills"
-Comment2 ""
+Comment2 "Schematic of the Futuwear V2 clothing main PCB"
 Comment3 ""
 Comment4 ""
@@
 $EndComp
 $Comp
-L +3.3V #PWR01
+L +3.3V #PWR22
 U 1 1 5971E3B1
 P 6625 1225
-F 0 "#PWR01" H 6625 1075 50  0001 C CNN
+F 0 "#PWR22" H 6625 1075 50  0001 C CNN
 F 1 "+3.3V" H 6625 1365 50  0000 C CNN
 F 2 "" H 6625 1225 50  0001 C CNN
@@
 $EndComp
 $Comp
-L GND #PWR02
+L GND #PWR16
 U 1 1 59720FC3
 P 4125 1350
-F 0 "#PWR02" H 4125 1100 50  0001 C CNN
+F 0 "#PWR16" H 4125 1100 50  0001 C CNN
 F 1 "GND" H 4125 1200 50  0000 C CNN
 F 2 "" H 4125 1350 50  0001 C CNN
@@
 LDO-Circuit\n
 $Comp
-L +3.3V #PWR03
+L +3.3V #PWR2
 U 1 1 59722043
 P 800 2850
-F 0 "#PWR03" H 800 2700 50  0001 C CNN
+F 0 "#PWR2" H 800 2700 50  0001 C CNN
 F 1 "+3.3V" H 800 2990 50  0000 C CNN
 F 2 "" H 800 2850 50  0001 C CNN
@@
 $EndComp
 $Comp
-L GND #PWR04
+L GND #PWR3
 U 1 1 5972240F
 P 800 3500
-F 0 "#PWR04" H 800 3250 50  0001 C CNN
+F 0 "#PWR3" H 800 3250 50  0001 C CNN
 F 1 "GND" H 800 3350 50  0000 C CNN
 F 2 "" H 800 3500 50  0001 C CNN
@@
 $EndComp
 $Comp
-L +3.3V #PWR05
+L +3.3V #PWR6
 U 1 1 59727C57
 P 2450 2700
-F 0 "#PWR05" H 2450 2550 50  0001 C CNN
+F 0 "#PWR6" H 2450 2550 50  0001 C CNN
 F 1 "+3.3V" H 2450 2840 50  0000 C CNN
 F 2 "" H 2450 2700 50  0001 C CNN
@@
 $EndComp
 $Comp
-L GND #PWR06
+L GND #PWR7
 U 1 1 597288AB
 P 2450 3600
-F 0 "#PWR06" H 2450 3350 50  0001 C CNN
+F 0 "#PWR7" H 2450 3350 50  0001 C CNN
 F 1 "GND" H 2450 3450 50  0000 C CNN
 F 2 "" H 2450 3600 50  0001 C CNN
@@
 CHIP_PU HIGH
 $Comp
-L GND #PWR07
+L GND #PWR23
 U 1 1 5972E666
 P 6640 5250
-F 0 "#PWR07" H 6640 5000 50  0001 C CNN
+F 0 "#PWR23" H 6640 5000 50  0001 C CNN
 F 1 "GND" H 6640 5100 50  0000 C CNN
 F 2 "" H 6640 5250 50  0001 C CNN
@@
 $EndComp
 $Comp
-L GND #PWR08
+L GND #PWR10
 U 1 1 597C0D8F
 P 2940 1640
-F 0 "#PWR08" H 2940 1390 50  0001 C CNN
+F 0 "#PWR10" H 2940 1390 50  0001 C CNN
 F 1 "GND" H 2940 1490 50  0000 C CNN
 F 2 "" H 2940 1640 50  0001 C CNN
@@
 $EndComp
 $Comp
-L GND #PWR09
+L GND #PWR1
 U 1 1 597CC4A0
 P 740 1670
-F 0 "#PWR09" H 740 1420 50  0001 C CNN
+F 0 "#PWR1" H 740 1420 50  0001 C CNN
 F 1 "GND" H 740 1520 50  0000 C CNN
 F 2 "" H 740 1670 50  0001 C CNN
@@
 $EndComp
 $Comp
-L GND #PWR010
+L GND #PWR5
 U 1 1 597D3152
 P 2400 1990
-F 0 "#PWR010" H 2400 1740 50  0001 C CNN
+F 0 "#PWR5" H 2400 1740 50  0001 C CNN
 F 1 "GND" H 2400 1840 50  0000 C CNN
 F 2 "" H 2400 1990 50  0001 C CNN
@@
 $EndComp
 $Comp
-L GND #PWR011
+L GND #PWR19
 U 1 1 5979BE1F
 P 6040 5830
-F 0 "#PWR011" H 6040 5580 50  0001 C CNN
+F 0 "#PWR19" H 6040 5580 50  0001 C CNN
 F 1 "GND" H 6040 5680 50  0000 C CNN
 F 2 "" H 6040 5830 50  0001 C CNN
@@
 $EndComp
 $Comp
-L +3.3V #PWR012
+L +3.3V #PWR21
 U 1 1 597F3871
 P 6600 3400
-F 0 "#PWR012" H 6600 3250 50  0001 C CNN
+F 0 "#PWR21" H 6600 3250 50  0001 C CNN
 F 1 "+3.3V" H 6600 3540 50  0000 C CNN
 F 2 "" H 6600 3400 50  0001 C CNN
@@
 $EndComp
 $Comp
-L +3.3V #PWR013
+L +3.3V #PWR24
 U 1 1 597F3ACF
 P 6900 3400
-F 0 "#PWR013" H 6900 3250 50  0001 C CNN
+F 0 "#PWR24" H 6900 3250 50  0001 C CNN
 F 1 "+3.3V" H 6900 3540 50  0000 C CNN
 F 2 "" H 6900 3400 50  0001 C CNN
@@
 NoConn ~ 9020 1480
 $Comp
-L +BATT #PWR014
+L +BATT #PWR32
 U 1 1 5984ACAC
 P 10755 1125
-F 0 "#PWR014" H 10755 975 50  0001 C CNN
+F 0 "#PWR32" H 10755 975 50  0001 C CNN
 F 1 "+BATT" H 10755 1265 50  0000 C CNN
 F 2 "" H 10755 1125 50  0001 C CNN
@@
 $EndComp
 $Comp
-L +BATT #PWR015
+L +BATT #PWR11
 U 1 1 5984CCC8
 P 3240 1135
-F 0 "#PWR015" H 3240 985 50  0001 C CNN
+F 0 "#PWR11" H 3240 985 50  0001 C CNN
 F 1 "+BATT" H 3240 1275 50  0000 C CNN
 F 2 "" H 3240 1135 50  0001 C CNN
@@
 GPIO14
 $Comp
-L PWR_FLAG #FLG016
+L PWR_FLAG #FLG1
 U 1 1 5988CE3F
 P 740 1230
-F 0 "#FLG016" H 740 1305 50  0001 C CNN
+F 0 "#FLG1" H 740 1305 50  0001 C CNN
 F 1 "PWR_FLAG" H 740 1380 50  0000 C CNN
 F 2 "" H 740 1230 50  0001 C CNN
@@
 $EndComp
 $Comp
-L +BATT #PWR017
+L +BATT #PWR15
 U 1 1 59896F9B
 P 3900 900
-F 0 "#PWR017" H 3900 750 50  0001 C CNN
+F 0 "#PWR15" H 3900 750 50  0001 C CNN
 F 1 "+BATT" H 3900 1040 50  0000 C CNN
 F 2 "" H 3900 900 50  0001 C CNN
@@
 -BATT
 $Comp
-L PWR_FLAG #FLG018
+L PWR_FLAG #FLG4
 U 1 1 598A5F92
 P 10520 1580
-F 0 "#FLG018" H 10520 1655 50  0001 C CNN
+F 0 "#FLG4" H 10520 1655 50  0001 C CNN
 F 1 "PWR_FLAG" H 10520 1730 50  0000 C CNN
 F 2 "" H 10520 1580 50  0001 C CNN
@@
 USB_IN
 $Comp
-L GND #PWR019
+L GND #PWR4
 U 1 1 598D6024
 P 1020 4750
-F 0 "#PWR019" H 1020 4500 50  0001 C CNN
+F 0 "#PWR4" H 1020 4500 50  0001 C CNN
 F 1 "GND" H 1020 4600 50  0000 C CNN
 F 2 "" H 1020 4750 50  0001 C CNN
@@
 GPIO16
 $Comp
-L PWR_FLAG #FLG020
+L PWR_FLAG #FLG2
 U 1 1 598467B7
 P 3240 1290
-F 0 "#FLG020" H 3240 1365 50  0001 C CNN
+F 0 "#FLG2" H 3240 1365 50  0001 C CNN
 F 1 "PWR_FLAG" H 3240 1440 50  0000 C CNN
 F 2 "" H 3240 1290 50  0001 C CNN
@@
 Text Label 4490 3900 2    47   ~ 0
 EN
-Text Label 6650 4850 0    47   ~ 0
+Text Label 7350 4850 0    47   ~ 0
 IO0
 $Comp
@@
 $EndComp
 $Comp
-L GND #PWR021
+L GND #PWR18
 U 1 1 598218AC
 P 5600 1375
-F 0 "#PWR021" H 5600 1125 50  0001 C CNN
+F 0 "#PWR18" H 5600 1125 50  0001 C CNN
 F 1 "GND" H 5600 1225 50  0000 C CNN
 F 2 "" H 5600 1375 50  0001 C CNN
@@
 NoConn ~ 9825 5775
 $Comp
-L GND #PWR022
+L GND #PWR31
 U 1 1 5982D96A
 P 9375 3425
-F 0 "#PWR022" H 9375 3175 50  0001 C CNN
+F 0 "#PWR31" H 9375 3175 50  0001 C CNN
 F 1 "GND" H 9375 3275 50  0000 C CNN
 F 2 "" H 9375 3425 50  0001 C CNN
@@
 $EndComp
 $Comp
-L GND #PWR023
+L GND #PWR28
 U 1 1 5982E7A6
 P 8925 4625
-F 0 "#PWR023" H 8925 4375 50  0001 C CNN
+F 0 "#PWR28" H 8925 4375 50  0001 C CNN
 F 1 "GND" H 8925 4475 50  0000 C CNN
 F 2 "" H 8925 4625 50  0001 C CNN
@@
 $EndComp
 $Comp
-L GND #PWR024
+L GND #PWR30
 U 1 1 59837BD7
 P 9050 6175
-F 0 "#PWR024" H 9050 5925 50  0001 C CNN
+F 0 "#PWR30" H 9050 5925 50  0001 C CNN
 F 1 "GND" H 9050 6025 50  0000 C CNN
 F 2 "" H 9050 6175 50  0001 C CNN
@@
 $EndComp
 $Comp
-L GND #PWR025
+L GND #PWR27
 U 1 1 5983B81C
 P 8675 5300
-F 0 "#PWR025" H 8675 5050 50  0001 C CNN
+F 0 "#PWR27" H 8675 5050 50  0001 C CNN
 F 1 "GND" H 8675 5150 50  0000 C CNN
 F 2 "" H 8675 5300 50  0001 C CNN
@@
 $EndComp
 $Comp
-L +3.3V #PWR026
+L +3.3V #PWR26
 U 1 1 59840AF6
 P 8675 4750
-F 0 "#PWR026" H 8675 4600 50  0001 C CNN
+F 0 "#PWR26" H 8675 4600 50  0001 C CNN
 F 1 "+3.3V" H 8675 4890 50  0000 C CNN
 F 2 "" H 8675 4750 50  0001 C CNN
@@
 GPIO18
 $Comp
-L GND #PWR027
+L GND #PWR14
 U 1 1 5984853F
 P 3675 7500
-F 0 "#PWR027" H 3675 7250 50  0001 C CNN
+F 0 "#PWR14" H 3675 7250 50  0001 C CNN
 F 1 "GND" H 3675 7350 50  0000 C CNN
 F 2 "" H 3675 7500 50  0001 C CNN
@@
 $EndComp
 $Comp
-L GND #PWR028
+L GND #PWR17
 U 1 1 5984A891
 P 4590 5150
-F 0 "#PWR028" H 4590 4900 50  0001 C CNN
+F 0 "#PWR17" H 4590 4900 50  0001 C CNN
 F 1 "GND" H 4590 5000 50  0000 C CNN
 F 2 "" H 4590 5150 50  0001 C CNN
@@
 $EndComp
 $Comp
-L GND #PWR029
+L GND #PWR20
 U 1 1 598649D1
 P 6595 2490
-F 0 "#PWR029" H 6595 2240 50  0001 C CNN
+F 0 "#PWR20" H 6595 2240 50  0001 C CNN
 F 1 "GND" H 6595 2340 50  0000 C CNN
 F 2 "" H 6595 2490 50  0001 C CNN
@@
 $EndComp
 $Comp
-L GND #PWR030
+L GND #PWR29
 U 1 1 59888474
 P 9005 1225
-F 0 "#PWR030" H 9005 975 50  0001 C CNN
+F 0 "#PWR29" H 9005 975 50  0001 C CNN
 F 1 "GND" H 9005 1075 50  0000 C CNN
 F 2 "" H 9005 1225 50  0001 C CNN
@@
 $EndComp
 $Comp
-L PWR_FLAG #FLG031
+L PWR_FLAG #FLG3
 U 1 1 5988D03E
 P 6330 2510
-F 0 "#FLG031" H 6330 2585 50  0001 C CNN
+F 0 "#FLG3" H 6330 2585 50  0001 C CNN
 F 1 "PWR_FLAG" H 6330 2660 50  0000 C CNN
 F 2 "" H 6330 2510 50  0001 C CNN
@@
 $EndComp
 $Comp
-L PWR_FLAG #FLG032
+L PWR_FLAG #FLG5
 U 1 1 59898C90
 P 10575 2505
-F 0 "#FLG032" H 10575 2580 50  0001 C CNN
+F 0 "#FLG5" H 10575 2580 50  0001 C CNN
 F 1 "PWR_FLAG" H 10575 2655 50  0000 C CNN
 F 2 "" H 10575 2505 50  0001 C CNN
@@
 	2245 1990 2400 1990
 Wire Wire Line
-	6490 4850 6650 4850
+	6490 4850 7350 4850
 Wire Wire Line
 	6040 5450 6040 5520
@@
 Connection ~ 10575 2440
 $Comp
-L +BATT #PWR033
+L +BATT #PWR8
 U 1 1 598A2C1F
 P 2525 4275
-F 0 "#PWR033" H 2525 4125 50  0001 C CNN
+F 0 "#PWR8" H 2525 4125 50  0001 C CNN
 F 1 "+BATT" H 2525 4415 50  0000 C CNN
 F 2 "" H 2525 4275 50  0001 C CNN
@@
 	3150 5250 3275 5250
 $Comp
-L GND #PWR034
+L GND #PWR12
 U 1 1 598BE5AB
 P 3550 6455
-F 0 "#PWR034" H 3550 6205 50  0001 C CNN
+F 0 "#PWR12" H 3550 6205 50  0001 C CNN
 F 1 "GND" H 3550 6305 50  0000 C CNN
 F 2 "" H 3550 6455 50  0001 C CNN
@@
 $EndComp
 $Comp
-L +3.3V #PWR035
+L +3.3V #PWR13
 U 1 1 598BEECD
 P 3575 6125
-F 0 "#PWR035" H 3575 5975 50  0001 C CNN
+F 0 "#PWR13" H 3575 5975 50  0001 C CNN
 F 1 "+3.3V" H 3575 6265 50  0000 C CNN
 F 2 "" H 3575 6125 50  0001 C CNN
 F 3 "" H 3575 6125 50  0001 C CNN
 	1    3575 6125
-	-1   0    0    1
+	1    0    0    -1
 $EndComp
 $Comp
@@
 $EndComp
 $Comp
-L GND #PWR036
+L GND #PWR9
 U 1 1 5996C51C
 P 2550 1550
-F 0 "#PWR036" H 2550 1300 50  0001 C CNN
+F 0 "#PWR9" H 2550 1300 50  0001 C CNN
 F 1 "GND" H 2550 1400 50  0000 C CNN
 F 2 "" H 2550 1550 50  0001 C CNN
@@
 Wire Wire Line
 	5800 1300 6625 1300
+$Comp
+L +3.3V #PWR25
+U 1 1 59A01036
+P 7200 4450
+F 0 "#PWR25" H 7200 4300 50  0001 C CNN
+F 1 "+3.3V" H 7200 4590 50  0000 C CNN
+F 2 "" H 7200 4450 50  0001 C CNN
+F 3 "" H 7200 4450 50  0001 C CNN
+	1    7200 4450
+	1    0    0    -1
+$EndComp
+$Comp
+L R_Small R19
+U 1 1 59A0170A
+P 7200 4650
+F 0 "R19" H 7230 4670 50  0000 L CNN
+F 1 "10kΩ" H 7230 4610 50  0000 L CNN
+F 2 "" H 7200 4650 50  0001 C CNN
+F 3 "" H 7200 4650 50  0001 C CNN
+	1    7200 4650
+	1    0    0    -1
+$EndComp
+Wire Wire Line
+	7200 4450 7200 4550
+Wire Wire Line
+	7200 4750 7200 4850
+Connection ~ 7200 4850
 $EndSCHEMATC
